File: pi0ii040/USB.kicad_sch (KiCad schematic)
At the start: 0 parts

Commit message: Add submodules, start schematic
Parts:
- added C_LDO1, C_LDO2: 1u, Capacitor_SMD:C_0402_1005Metric, symbol Device:C_Small
- added C_Shield1: 4.7n, Capacitor_SMD:C_0402_1005Metric, symbol Device:C_Small
- added F1: 500mA, Fuse:Fuse_0805_2012Metric, symbol Device:Polyfuse_Small
- added J1: SM04B, Connector_JST:JST_SH_SM04B-SRSS-TB_1x04-1MP_P1.00mm_Horizontal, symbol Connector:Conn_01x04_Female
- added R_Shield1: 1M, Resistor_SMD:R_0402_1005Metric, symbol Device:R_Small
- added R_USB1, R_USB2: 5k1, Resistor_SMD:R_0402_1005Metric, symbol Device:R_Small
- added U3: PRTR5V0U2X, random-keyboard-parts:SOT143B, symbol cipulot_parts:PRTR5V0U2X
- added U4: XC6206PxxxMR, Package_TO_SOT_SMD:SOT-23, symbol Regulator_Linear:XC6206PxxxMR
- added USB1: HRO-TYPE-C-31-M-12, cipulot_parts:HRO-TYPE-C-31-M-12-Assembly, symbol cipulot_parts:HRO-TYPE-C-31-M-12
Connections:
- new net: R_USB2.1, USB1.10 (CC2)
- new net: R_USB1.1, USB1.4 (CC1)
- new net +3V3: C_LDO2.1, U4.2 (VO)
- new net +5V: C_LDO1.1, F1.2, J1.1 (Pin_1), U4.3 (VI)
- new net D+: J1.3 (Pin_3), U3.2 (IO1), USB1.6 (DP1), USB1.8 (DP2)
- new net D-: J1.2 (Pin_2), U3.3 (IO2), USB1.5 (DN2), USB1.7 (DN1)
- new net GND: C_LDO1.2, C_LDO2.2, C_Shield1.1, J1.4 (Pin_4), R_Shield1.2, R_USB1.2, R_USB2.2, U3.1 (GND), U4.1 (GND), USB1.1 (GND), USB1.12 (GND)
- new net GNDREF: C_Shield1.2, R_Shield1.1, USB1.13 (SHIELD)
- new net VCC: F1.1, U3.4 (VCC), USB1.11 (VBUS), USB1.2 (VBUS)
- no-connect marks 0 -> 2
Other:
- note added: "ESD, Power Regulation & Protection"
- note added: "Shielding"
- note added: "USB & JST"
