File: pi0ii040/MCU.kicad_sch (KiCad schematic)
At the start: 0 parts

Commit message: Add submodules, start schematic
Parts:
- added C_1V-Decoup1, C_3V-Decoup2: 1u, Capacitor_SMD:C_0402_1005Metric, symbol Device:C_Small
- added C_1V-Decoup2, C_1V-Decoup3, C_3V-Decoup3, C_3V-Decoup4, C_3V-Decoup5, C_3V-Decoup6, C_3V-Decoup7, C_3V-Decoup8, C_3V-Decoup9, C_Flash1: .1u, Capacitor_SMD:C_0402_1005Metric, symbol Device:C_Small
- added C_3V-Decoup1: 10u, Capacitor_SMD:C_0402_1005Metric, symbol Device:C_Small
- added C_Crystal1, C_Crystal2: 22pF, Capacitor_SMD:C_0402_1005Metric, symbol Device:C_Small
- added R_Crystal1, R_Flash1, R_RST1: 1k, Resistor_SMD:R_0402_1005Metric, symbol Device:R_Small
- added R_DATA1, R_DATA2: 27, Resistor_SMD:R_0402_1005Metric, symbol Device:R_Small
- added SW1: Reset, Connector_PinHeader_1.27mm:PinHeader_1x02_P1.27mm_Vertical, symbol Switch:SW_Push
- added U1: W25Q128JVS, Package_SO:SOIC-8_5.23x5.23mm_P1.27mm, symbol Memory_Flash:W25Q128JVS
- added U2: RP2040, Package_DFN_QFN:QFN-56-1EP_7x7mm_P0.4mm_EP3.2x3.2mm, symbol MCU_RaspberryPi:RP2040
- added Y1: 12MHz, Crystal:Crystal_SMD_3225-4Pin_3.2x2.5mm, symbol Device:Crystal_GND24_Small
Connections:
- new net: R_DATA2.2, U2.46 (USB_DM)
- new net: R_DATA1.2, U2.47 (USB_DP)
- new net: C_Crystal2.2, R_Crystal1.1, Y1.1
- new net: R_Flash1.1, SW1.2
- new net +1V1: C_1V-Decoup1.1, C_1V-Decoup2.1, C_1V-Decoup3.1, U2.23 (DVDD), U2.45 (VREG_VOUT), U2.50 (DVDD)
- new net +3V3: C_3V-Decoup1.1, C_3V-Decoup2.1, C_3V-Decoup3.1, C_3V-Decoup4.1, C_3V-Decoup5.1, C_3V-Decoup6.1, C_3V-Decoup7.1, C_3V-Decoup8.1, C_3V-Decoup9.1, C_Flash1.1, R_RST1.1, U1.8 (VCC), U2.1 (IOVDD), U2.10 (IOVDD), U2.22 (IOVDD), U2.33 (IOVDD), U2.42 (IOVDD), U2.43 (ADC_AVDD), U2.44 (VREG_IN), U2.48 (USB_VDD), U2.49 (IOVDD)
- new net CS: R_Flash1.2, U1.1 (~{CS}), U2.56 (QSPI_SS)
- new net D+: R_DATA1.1
- new net D-: R_DATA2.1
- new net GND: C_1V-Decoup1.2, C_1V-Decoup2.2, C_1V-Decoup3.2, C_3V-Decoup1.2, C_3V-Decoup2.2, C_3V-Decoup3.2, C_3V-Decoup4.2, C_3V-Decoup5.2, C_3V-Decoup6.2, C_3V-Decoup7.2, C_3V-Decoup8.2, C_3V-Decoup9.2, C_Crystal1.1, C_Crystal2.1, C_Flash1.2, SW1.1, U1.4 (GND), U2.19 (TESTEN), U2.57 (GND), Y1.2, Y1.4
- new net QSPI_CLK: U1.6 (CLK), U2.52 (QSPI_SCLK)
- new net RESET: R_RST1.2, U2.26 (RUN)
- new net SD0: U1.5 (DI(IO0)), U2.53 (QSPI_SD0)
- new net SD1: U1.2 (DO(IO1)), U2.55 (QSPI_SD1)
- new net SD2: U1.3 (IO2), U2.54 (QSPI_SD2)
- new net SD3: U1.7 (IO3), U2.51 (QSPI_SD3)
- new net SWCLK: U2.24 (SWCLK)
- new net SWDIO: U2.25 (SWD)
- new net XTAL_IN: C_Crystal1.2, U2.20 (XIN), Y1.3
- new net XTAL_OUT: R_Crystal1.2, U2.21 (XOUT)
- new net col0: U2.32 (GPIO21)
- new net col1: U2.7 (GPIO5)
- new net col10: U2.15 (GPIO12)
- new net col11: U2.14 (GPIO11)
- new net col2: U2.6 (GPIO4)
- new net col3: U2.5 (GPIO3)
- new net col4: U2.4 (GPIO2)
- new net col5: U2.3 (GPIO1)
- new net col6: U2.2 (GPIO0)
- new net col7: U2.18 (GPIO15)
- new net col8: U2.17 (GPIO14)
- new net col9: U2.16 (GPIO13)
- new net row0: U2.40 (GPIO28_ADC2)
- new net row1: U2.39 (GPIO27_ADC1)
- new net row2: U2.31 (GPIO20)
- new net row3: U2.8 (GPIO6)
Other:
- note added: "1V1 Decoupling"
- note added: "3V3 Decoupling"
- note added: "Crystal"
- note added: "Flash"
- note added: "MCU"

Commit message: Finish? pcb
Parts:
- removed U2: RP2040, Package_DFN_QFN:QFN-56-1EP_7x7mm_P0.4mm_EP3.2x3.2mm, symbol MCU_RaspberryPi:RP2040
- added U1: RP2040, cipulot_parts:RP2040-QFN-56, symbol cipulot_parts:RP2040
- renumbered U1 to U2
Connections:
- net +1V1: now also U1.23 (DVDD), U1.45 (VREG_VOUT), U1.50 (DVDD)
- net +3V3: now also U1.1 (IOVDD), U1.10 (IOVDD), U1.22 (IOVDD), U1.33 (IOVDD), U1.42 (IOVDD), U1.43 (ADC_AVDD), U1.44 (VREG_VIN), U1.48 (USB_VDD), U1.49 (IOVDD)
- net CS: now also U1.56 (QSPI_SS_N)
- net GND: now also U1.19 (TESTEN), U1.57 (GND)
- net QSPI_CLK: now also U1.52 (QSPI_SCLK)
- net RESET: now also U1.26 (~{RUN})
- net SD0: now also U1.53 (QSPI_SD0)
- net SD1: now also U1.55 (QSPI_SD1)
- net SD2: now also U1.54 (QSPI_SD2)
- net SD3: now also U1.51 (QSPI_SD3)
- net SWCLK: now also U1.24 (SWCLK)
- net SWDIO: now also U1.25 (SWDIO)
- net XTAL_IN: now also U1.20 (XTAL_IN)
- net XTAL_OUT: now also U1.21 (XTAL_OUT)
- net col0: now also U1.32 (GPIO21)
- net col1: now also U1.5 (GPIO3)
- net col10: now also U1.15 (GPIO12)
- net col11: now also U1.14 (GPIO11)
- net col2: now also U1.6 (GPIO4)
- net col3: now also U1.7 (GPIO5)
- net col4: now also U1.4 (GPIO2)
- net col5: now also U1.3 (GPIO1)
- net col6: now also U1.2 (GPIO0)
- net col7: now also U1.18 (GPIO15)
- net col8: now also U1.17 (GPIO14)
- net col9: now also U1.16 (GPIO13)
- net row0: now also U1.40 (GPIO28/ADC2)
- net row1: now also U1.39 (GPIO27/ADC1)
- net row2: now also U1.31 (GPIO20)
- net row3: now also U1.29 (GPIO18)
- net at R_DATA2.2: now also U1.46 (D-)
- net at R_DATA1.2: now also U1.47 (D+)
