File: pi0ii040/Misc.kicad_sch (KiCad schematic)
At the start: 0 parts

Commit message: Finish? pcb
Parts:
- added H1: PCB Outline, M0ii040関連KaWaii40:m0ii040_PCB_Template_v1.0.1, symbol Mechanical:MountingHole_Pad
- added J2: SWD, Connector_PinHeader_2.54mm:PinHeader_1x05_P2.54mm_Vertical, symbol Connector:Conn_01x05_Female
Connections:
- new net +3V3: J2.2 (Pin_2)
- new net GND: H1.1, J2.3 (Pin_3)
- new net RESET: J2.1 (Pin_1)
- new net SWCLK: J2.5 (Pin_5)
- new net SWDIO: J2.4 (Pin_4)
Other:
- note added: "Connectors"
Changed lines of the file:
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@@
 (kicad_sch (version 20230121) (generator eeschema)
   (paper "A4")
+  (polyline (pts (xy 12.7 12.7) (xy 12.7 31.75))
+    (stroke (width 0) (type default))
+  )
+  (wire (pts (xy 40.005 22.225) (xy 51.435 22.225))
+    (stroke (width 0) (type default))
+  )
+  (wire (pts (xy 40.005 19.685) (xy 51.435 19.685))
+    (stroke (width 0) (type default))
+  )
+  (polyline (pts (xy 64.135 12.7) (xy 64.135 31.75))
+    (stroke (width 0) (type default))
+  )
+  (polyline (pts (xy 43.815 31.75) (xy 64.135 31.75))
+    (stroke (width 0) (type default))
+  )
+  (polyline (pts (xy 12.7 31.75) (xy 44.45 31.75))
+    (stroke (width 0) (type default))
+  )
+  (polyline (pts (xy 12.7 12.7) (xy 64.135 12.7))
+    (stroke (width 0) (type default))
+  )
+  (text "Connectors\n" (at 13.335 15.24 0)
+    (effects (font (size 1.27 1.27)) (justify left bottom))
+  )
+  (global_label "RESET" (shape input) (at 51.435 17.145 180) (fields_autoplaced)
+    (effects (font (size 1.27 1.27)) (justify right))
+    (property "Intersheetrefs" "${INTERSHEET_REFS}" (at 43.2767 17.0656 0)
+      (effects (font (size 1.27 1.27)) (justify right) hide)
+    )
+  )
+  (global_label "SWDIO" (shape input) (at 51.435 24.765 180) (fields_autoplaced)
+    (effects (font (size 1.27 1.27)) (justify right))
+    (property "Intersheetrefs" "${INTERSHEET_REFS}" (at 43.1557 24.6856 0)
+      (effects (font (size 1.27 1.27)) (justify right) hide)
+    )
+  )
+  (global_label "SWCLK" (shape input) (at 51.435 27.305 180) (fields_autoplaced)
+    (effects (font (size 1.27 1.27)) (justify right))
+    (property "Intersheetrefs" "${INTERSHEET_REFS}" (at 42.7929 27.2256 0)
+      (effects (font (size 1.27 1.27)) (justify right) hide)
+    )
+  )
+  (symbol (lib_id "power:GND") (at 17.145 24.765 0) (unit 1)
+    (in_bom yes) (on_board yes) (dnp no) (fields_autoplaced)
+    (property "Reference" "#PWR038" (at 17.145 31.115 0)
+      (effects (font (size 1.27 1.27)) hide)
+    )
+    (property "Value" "GND" (at 17.145 29.21 0)
+      (effects (font (size 1.27 1.27)))
+    )
+    (property "Footprint" "" (at 17.145 24.765 0)
+      (effects (font (size 1.27 1.27)) hide)
+    )
+    (property "Datasheet" "" (at 17.145 24.765 0)
+      (effects (font (size 1.27 1.27)) hide)
+    )
+    (pin "1")
+    (instances
+      (project "pi0ii040"
+        (path "/b030bddc-56a8-497a-8df3-ec17c8e3ece5/2fbf78f8-73f0-4f62-afa7-da3d07a42383"
+          (reference "#PWR038") (unit 1)
+        )
+      )
+      (project "SST60"
+        (path "/e63e39d7-6ac0-4ffd-8aa3-1841a4541b55/4eb096de-f3a2-4165-be7d-6a3944b02fe7"
+          (reference "#PWR0141") (unit 1)
+        )
+      )
+    )
+  )
+  (symbol (lib_id "power:GND") (at 40.005 22.225 0) (unit 1)
+    (in_bom yes) (on_board yes) (dnp no)
+    (property "Reference" "#PWR037" (at 40.005 28.575 0)
+      (effects (font (size 1.27 1.27)) hide)
+    )
+    (property "Value" "GND" (at 40.005 26.035 0)
+      (effects (font (size 1.27 1.27)))
+    )
+    (property "Footprint" "" (at 40.005 22.225 0)
+      (effects (font (size 1.27 1.27)) hide)
+    )
+    (property "Datasheet" "" (at 40.005 22.225 0)
+      (effects (font (size 1.27 1.27)) hide)
+    )
+    (pin "1")
+    (instances
+      (project "pi0ii040"
+        (path "/b030bddc-56a8-497a-8df3-ec17c8e3ece5/2fbf78f8-73f0-4f62-afa7-da3d07a42383"
+          (reference "#PWR037") (unit 1)
+        )
+      )
+      (project "SST60"
+        (path "/e63e39d7-6ac0-4ffd-8aa3-1841a4541b55/4eb096de-f3a2-4165-be7d-6a3944b02fe7"
+          (reference "#PWR0139") (unit 1)
+        )
+      )
+    )
+  )
+  (symbol (lib_id "Connector:Conn_01x05_Female") (at 56.515 22.225 0) (unit 1)
+    (in_bom yes) (on_board yes) (dnp no) (fields_autoplaced)
+    (property "Reference" "J2" (at 57.785 20.9549 0)
+      (effects (font (size 1.27 1.27)) (justify left))
+    )
+    (property "Value" "SWD" (at 57.785 23.4949 0)
+      (effects (font (size 1.27 1.27)) (justify left))
+    )
+    (property "Footprint" "Connector_PinHeader_2.54mm:PinHeader_1x05_P2.54mm_Vertical" (at 56.515 22.225 0)
+      (effects (font (size 1.27 1.27)) hide)
+    )
+    (property "Datasheet" "~" (at 56.515 22.225 0)
+      (effects (font (size 1.27 1.27)) hide)
+    )
+    (pin "1")
+    (pin "2")
+    (pin "3")
+    (pin "4")
+    (pin "5")
+    (instances
+      (project "pi0ii040"
+        (path "/b030bddc-56a8-497a-8df3-ec17c8e3ece5/2fbf78f8-73f0-4f62-afa7-da3d07a42383"
+          (reference "J2") (unit 1)
+        )
+      )
+      (project "SST60"
+        (path "/e63e39d7-6ac0-4ffd-8aa3-1841a4541b55/4eb096de-f3a2-4165-be7d-6a3944b02fe7"
+          (reference "J2") (unit 1)
+        )
+      )
+    )
+  )
+  (symbol (lib_id "power:+3V3") (at 40.005 19.685 0) (unit 1)
+    (in_bom yes) (on_board yes) (dnp no)
+    (property "Reference" "#PWR036" (at 40.005 23.495 0)
+      (effects (font (size 1.27 1.27)) hide)
+    )
+    (property "Value" "+3V3" (at 40.005 15.24 0)
+      (effects (font (size 1.27 1.27)))
+    )
+    (property "Footprint" "" (at 40.005 19.685 0)
+      (effects (font (size 1.27 1.27)) hide)
+    )
+    (property "Datasheet" "" (at 40.005 19.685 0)
+      (effects (font (size 1.27 1.27)) hide)
+    )
+    (pin "1")
+    (instances
+      (project "pi0ii040"
+        (path "/b030bddc-56a8-497a-8df3-ec17c8e3ece5/2fbf78f8-73f0-4f62-afa7-da3d07a42383"
+          (reference "#PWR036") (unit 1)
+        )
+      )
+      (project "SST60"
+        (path "/e63e39d7-6ac0-4ffd-8aa3-1841a4541b55/4eb096de-f3a2-4165-be7d-6a3944b02fe7"
+          (reference "#PWR0140") (unit 1)
+        )
+      )
+    )
+  )
+  (symbol (lib_id "Mechanical:MountingHole_Pad") (at 17.145 22.225 0) (unit 1)
+    (in_bom yes) (on_board yes) (dnp no) (fields_autoplaced)
+    (property "Reference" "H1" (at 20.32 19.6849 0)
+      (effects (font (size 1.27 1.27)) (justify left))
+    )
+    (property "Value" "PCB Outline" (at 20.32 22.2249 0)
+      (effects (font (size 1.27 1.27)) (justify left))
+    )
+    (property "Footprint" "M0ii040関連KaWaii40:m0ii040_PCB_Template_v1.0.1" (at 17.145 22.225 0)
+      (effects (font (size 1.27 1.27)) hide)
+    )
+    (property "Datasheet" "~" (at 17.145 22.225 0)
+      (effects (font (size 1.27 1.27)) hide)
+    )
+    (pin "1")
+    (instances
+      (project "pi0ii040"
+        (path "/b030bddc-56a8-497a-8df3-ec17c8e3ece5/2fbf78f8-73f0-4f62-afa7-da3d07a42383"
+          (reference "H1") (unit 1)
+        )
+      )
+      (project "SST60"
+        (path "/e63e39d7-6ac0-4ffd-8aa3-1841a4541b55/4eb096de-f3a2-4165-be7d-6a3944b02fe7"
+          (reference "H1") (unit 1)
+        )
+      )
+    )
+  )
 )
