File: pi0ii040/pi0ii040.kicad_pcb (KiCad board)
At the start: 2 copper layers, 228.6 x 76.2 mm, 1 part

Commit message: Finish? pcb
Parts:
- removed the REF** at (46.7, 75.5)
- added C_1V-Decoup1: 1u, Capacitor_SMD:C_0402_1005Metric, B.Cu at (54.9, 94.7)
- added C_1V-Decoup2: .1u, Capacitor_SMD:C_0402_1005Metric, B.Cu at (59.6, 93.0)
- added C_1V-Decoup3: .1u, Capacitor_SMD:C_0402_1005Metric, B.Cu at (55.3, 110.2)
- added C_3V-Decoup1: 10u, Capacitor_SMD:C_0402_1005Metric, B.Cu at (39.5, 75.3)
- added C_3V-Decoup2: 1u, Capacitor_SMD:C_0402_1005Metric, B.Cu at (53.7, 95.8)
- added C_3V-Decoup3: .1u, Capacitor_SMD:C_0402_1005Metric, B.Cu at (58.2, 92.2)
- added C_3V-Decoup4: .1u, Capacitor_SMD:C_0402_1005Metric, B.Cu at (51.0, 100.5)
- added C_3V-Decoup5: .1u, Capacitor_SMD:C_0402_1005Metric, B.Cu at (51.0, 99.5)
- added C_3V-Decoup6: .1u, Capacitor_SMD:C_0402_1005Metric, B.Cu at (62.7, 98.9)
- added C_3V-Decoup7: .1u, Capacitor_SMD:C_0402_1005Metric, B.Cu at (51.0, 98.5)
- added C_3V-Decoup8: .1u, Capacitor_SMD:C_0402_1005Metric, B.Cu at (56.5, 110.2)
- added C_3V-Decoup9: .1u, Capacitor_SMD:C_0402_1005Metric, B.Cu at (64.2, 104.9)
- added C_Crystal1: 22pF, Capacitor_SMD:C_0402_1005Metric, B.Cu at (61.7, 113.2)
- added C_Crystal2: 22pF, Capacitor_SMD:C_0402_1005Metric, B.Cu at (55.9, 113.1)
- added C_Flash1: .1u, Capacitor_SMD:C_0402_1005Metric, B.Cu at (66.6, 93.2)
- added C_LDO1: 1u, Capacitor_SMD:C_0402_1005Metric, B.Cu at (41.7, 70.2)
- added C_LDO2: 1u, Capacitor_SMD:C_0402_1005Metric, B.Cu at (39.4, 74.2)
- added C_Shield1: 4.7n, Capacitor_SMD:C_0402_1005Metric, B.Cu at (56.4, 56.7)
- added D1: D_Small, Diode_SMD:D_SOD-123, B.Cu at (29.8, 66.9)
- added D10: D_Small, Diode_SMD:D_SOD-123, B.Cu at (217.4, 66.9)
- added D11: D_Small, Diode_SMD:D_SOD-123, B.Cu at (236.5, 66.9)
- added D12: D_Small, Diode_SMD:D_SOD-123, B.Cu at (255.5, 66.9)
- added D13: D_Small, Diode_SMD:D_SOD-123, B.Cu at (48.3, 85.9)
- added D14: D_Small, Diode_SMD:D_SOD-123, B.Cu at (53.6, 85.9)
- added D15: D_Small, Diode_SMD:D_SOD-123, B.Cu at (88.8, 85.9)
- added D16: D_Small, Diode_SMD:D_SOD-123, B.Cu at (107.9, 85.9)
- added D17: D_Small, Diode_SMD:D_SOD-123, B.Cu at (126.9, 85.9)
- added D18: D_Small, Diode_SMD:D_SOD-123, B.Cu at (146.0, 85.9)
- added D19: D_Small, Diode_SMD:D_SOD-123, B.Cu at (165.0, 85.9)
- added D2: D_Small, Diode_SMD:D_SOD-123, B.Cu at (65.0, 66.9)
- added D20: D_Small, Diode_SMD:D_SOD-123, B.Cu at (184.1, 85.9)
- added D21: D_Small, Diode_SMD:D_SOD-123, B.Cu at (203.1, 85.9)
- added D22: D_Small, Diode_SMD:D_SOD-123, B.Cu at (222.2, 85.9)
- added D23: D_Small, Diode_SMD:D_SOD-123, B.Cu at (248.4, 85.9)
- added D24: D_Small, Diode_SMD:D_SOD-123, B.Cu at (36.9, 105.0)
- added D25: D_Small, Diode_SMD:D_SOD-123, B.Cu at (79.3, 105.0)
- added D26: D_Small, Diode_SMD:D_SOD-123, B.Cu at (98.3, 105.0)
- added D27: D_Small, Diode_SMD:D_SOD-123, B.Cu at (117.4, 105.0)
- added D28: D_Small, Diode_SMD:D_SOD-123, B.Cu at (136.4, 105.0)
- added D29: D_Small, Diode_SMD:D_SOD-123, B.Cu at (155.5, 105.0)
- added D3: D_Small, Diode_SMD:D_SOD-123, B.Cu at (84.1, 66.9)
- added D30: D_Small, Diode_SMD:D_SOD-123, B.Cu at (174.5, 105.0)
- added D31: D_Small, Diode_SMD:D_SOD-123, B.Cu at (193.6, 105.0)
- added D32: D_Small, Diode_SMD:D_SOD-123, B.Cu at (212.6, 105.0)
- added D33: D_Small, Diode_SMD:D_SOD-123, B.Cu at (234.1, 105.0)
- added D34: D_Small, Diode_SMD:D_SOD-123, B.Cu at (255.5, 105.0)
- added D35: D_Small, Diode_SMD:D_SOD-123, B.Cu at (72.1, 124.0)
- added D36: D_Small, Diode_SMD:D_SOD-123, B.Cu at (91.2, 124.0)
- added D37: D_Small, Diode_SMD:D_SOD-123, B.Cu at (129.3, 124.0)
- added D38: D_Small, Diode_SMD:D_SOD-123, B.Cu at (176.9, 124.0)
- added D39: D_Small, Diode_SMD:D_SOD-123, B.Cu at (210.3, 124.0)
- added D4: D_Small, Diode_SMD:D_SOD-123, B.Cu at (103.1, 66.9)
- added D40: D_Small, Diode_SMD:D_SOD-123, B.Cu at (231.7, 124.0)
- added D5: D_Small, Diode_SMD:D_SOD-123, B.Cu at (122.2, 66.9)
- added D6: D_Small, Diode_SMD:D_SOD-123, B.Cu at (141.2, 66.9)
- added D7: D_Small, Diode_SMD:D_SOD-123, B.Cu at (160.3, 66.9)
- added D8: D_Small, Diode_SMD:D_SOD-123, B.Cu at (179.3, 66.9)
- added D9: D_Small, Diode_SMD:D_SOD-123, B.Cu at (198.4, 66.9)
- added F1: 500mA, Fuse:Fuse_0805_2012Metric, B.Cu at (41.8, 68.0)
- added H1: PCB Outline, M0ii040関連KaWaii40:m0ii040_PCB_Template_v1.0.1, F.Cu at (37.9, 64.9)
- added J1: SM04B, Connector_JST:JST_SH_SM04B-SRSS-TB_1x04-1MP_P1.00mm_Horizontal, B.Cu at (54.9, 73.7)
- added J2: SWD, Connector_PinHeader_2.54mm:PinHeader_1x05_P2.54mm_Vertical, B.Cu at (30.5, 87.5)
- added MX1: MX-NoLED, MX_Only:MXOnly-1U-NoLED, F.Cu at (37.9, 64.9)
- added MX10: MX-NoLED, MX_Only:MXOnly-1U-NoLED, F.Cu at (209.3, 64.9)
- added MX11: MX-NoLED, MX_Only:MXOnly-1U-NoLED, F.Cu at (228.4, 64.9)
- added MX12: MX-NoLED, MX_Only:MXOnly-1U-NoLED, F.Cu at (247.4, 64.9)
- added MX13: MX-NoLED, MX_Only:MXOnly-1.25U-NoLED, F.Cu at (40.2, 83.9)
- added MX14: MX-NoLED, MX_Only:MXOnly-1U-NoLED, F.Cu at (61.7, 83.9)
- added MX15: MX-NoLED, MX_Only:MXOnly-1U-NoLED, F.Cu at (80.7, 83.9)
- added MX16: MX-NoLED, MX_Only:MXOnly-1U-NoLED, F.Cu at (99.8, 83.9)
- added MX17: MX-NoLED, MX_Only:MXOnly-1U-NoLED, F.Cu at (118.8, 83.9)
- added MX18: MX-NoLED, MX_Only:MXOnly-1U-NoLED, F.Cu at (137.9, 83.9)
- added MX19: MX-NoLED, MX_Only:MXOnly-1U-NoLED, F.Cu at (156.9, 83.9)
- added MX2: MX-NoLED, MX_Only:MXOnly-1U-NoLED, F.Cu at (56.9, 64.9)
- added MX20: MX-NoLED, MX_Only:MXOnly-1U-NoLED, F.Cu at (176.0, 83.9)
- added MX21: MX-NoLED, MX_Only:MXOnly-1U-NoLED, F.Cu at (195.0, 83.9)
- added MX22: MX-NoLED, MX_Only:MXOnly-1U-NoLED, F.Cu at (214.1, 83.9)
- added MX23: MX-NoLED, MX_Only:MXOnly-1.75U-NoLED, F.Cu at (240.3, 83.9)
- added MX24: MX-NoLED, MX_Only:MXOnly-1.75U-NoLED, F.Cu at (45.0, 103.0)
- added MX25: MX-NoLED, MX_Only:MXOnly-1U-NoLED, F.Cu at (71.2, 103.0)
- added MX26: MX-NoLED, MX_Only:MXOnly-1U-NoLED, F.Cu at (90.2, 103.0)
- added MX27: MX-NoLED, MX_Only:MXOnly-1U-NoLED, F.Cu at (109.3, 103.0)
- added MX28: MX-NoLED, MX_Only:MXOnly-1U-NoLED, F.Cu at (128.3, 103.0)
- added MX29: MX-NoLED, MX_Only:MXOnly-1U-NoLED, F.Cu at (147.4, 103.0)
- added MX3: MX-NoLED, MX_Only:MXOnly-1U-NoLED, F.Cu at (76.0, 64.9)
- added MX30: MX-NoLED, MX_Only:MXOnly-1U-NoLED, F.Cu at (166.4, 103.0)
- added MX31: MX-NoLED, MX_Only:MXOnly-1U-NoLED, F.Cu at (185.5, 103.0)
- added MX32: MX-NoLED, MX_Only:MXOnly-1U-NoLED, F.Cu at (204.5, 103.0)
- added MX33: MX-NoLED, MX_Only:MXOnly-1.25U-NoLED, F.Cu at (226.0, 103.0)
- added MX33: MX-NoLED, MX_Only:MXOnly-1U-NoLED, F.Cu at (223.6, 103.0)
- added MX34: MX-NoLED, MX_Only:MXOnly-1.25U-NoLED, F.Cu at (245.0, 103.0)
- added MX34: MX-NoLED, MX_Only:MXOnly-1U-NoLED, F.Cu at (247.4, 103.0)
- added MX35: MX-NoLED, MX_Only:MXOnly-1.25U-NoLED, F.Cu at (64.0, 122.0)
- added MX35: MX-NoLED, MX_Only:MXOnly-1U-NoLED, F.Cu at (61.7, 122.0)
- added MX36: MX-NoLED, MX_Only:MXOnly-1.25U-NoLED, F.Cu at (83.1, 122.0)
- added MX37: MX-NoLED, MX_Only:MXOnly-7U-ReversedStabilizers-NoLED, F.Cu at (142.6, 122.0)
- added MX37: MX-NoLED, MX_Only:MXOnly-2.75U-ReversedStabilizers-NoLED, F.Cu at (121.2, 122.0)
- added MX38: MX-NoLED, MX_Only:MXOnly-2.25U-ReversedStabilizers-NoLED, F.Cu at (168.8, 122.0)
- added MX39: MX-NoLED, MX_Only:MXOnly-1.25U-NoLED, F.Cu at (202.2, 122.0)
- added MX4: MX-NoLED, MX_Only:MXOnly-1U-NoLED, F.Cu at (95.0, 64.9)
- added MX40: MX-NoLED, MX_Only:MXOnly-1.25U-NoLED, F.Cu at (221.2, 122.0)
- added MX40: MX-NoLED, MX_Only:MXOnly-1U-NoLED, F.Cu at (223.6, 122.0)
- added MX5: MX-NoLED, MX_Only:MXOnly-1U-NoLED, F.Cu at (114.1, 64.9)
- added MX6: MX-NoLED, MX_Only:MXOnly-1U-NoLED, F.Cu at (133.1, 64.9)
- added MX7: MX-NoLED, MX_Only:MXOnly-1U-NoLED, F.Cu at (152.2, 64.9)
- added MX8: MX-NoLED, MX_Only:MXOnly-1U-NoLED, F.Cu at (171.2, 64.9)
- added MX9: MX-NoLED, MX_Only:MXOnly-1U-NoLED, F.Cu at (190.3, 64.9)
- added REF**: MountingHole_2.2mm_M2, MountingHole:MountingHole_2.2mm_M2, F.Cu at (74.0, 112.9)
- added REF**: MountingHole_2.2mm_M2, MountingHole:MountingHole_2.2mm_M2, F.Cu at (147.5, 93.3)
- added REF**: MountingHole_2.2mm_M2, MountingHole:MountingHole_2.2mm_M2, F.Cu at (208.8, 113.4)
- added REF**: MountingHole_2.2mm_M2, MountingHole:MountingHole_2.2mm_M2, F.Cu at (218.9, 74.2)
- added REF**: MountingHole_2.2mm_M2, MountingHole:MountingHole_2.2mm_M2, F.Cu at (71.2, 74.9)
- added R_Crystal1: 1k, Resistor_SMD:R_0402_1005Metric, B.Cu at (57.7, 110.2)
- added R_DATA1: 27, Resistor_SMD:R_0402_1005Metric, B.Cu at (57.1, 94.1)
- added R_DATA2: 27, Resistor_SMD:R_0402_1005Metric, B.Cu at (56.0, 94.1)
- added R_Flash1: 1k, Resistor_SMD:R_0402_1005Metric, B.Cu at (68.5, 83.0)
- added R_RST1: 1k, Resistor_SMD:R_0402_1005Metric, B.Cu at (33.4, 88.5)
- added R_Shield1: 1M, Resistor_SMD:R_0402_1005Metric, B.Cu at (55.2, 56.7)
- added R_USB1: 5k1, Resistor_SMD:R_0402_1005Metric, B.Cu at (45.5, 62.9)
- added R_USB2: 5k1, Resistor_SMD:R_0402_1005Metric, B.Cu at (49.7, 62.5)
- added SW1: Reset, Connector_PinHeader_1.27mm:PinHeader_1x02_P1.27mm_Vertical, B.Cu at (69.8, 80.0)
- added U1: RP2040, cipulot_parts:RP2040-QFN-56, B.Cu at (57.6, 102.4)
- added U2: W25Q128JVS, Package_SO:SOIC-8_5.23x5.23mm_P1.27mm, B.Cu at (70.3, 90.1)
- added U3: PRTR5V0U2X, random-keyboard-parts:SOT143B, B.Cu at (47.5, 67.3)
- added U4: XC6206PxxxMR, Package_TO_SOT_SMD:SOT-23, B.Cu at (42.3, 72.8)
- added USB1: HRO-TYPE-C-31-M-12, cipulot_parts:HRO-TYPE-C-31-M-12-Assembly, B.Cu at (47.4, 52.4)
- added Y1: 12MHz, Crystal:Crystal_SMD_3225-4Pin_3.2x2.5mm, B.Cu at (58.8, 113.0)
Routing:
- net row0: track 0.00 -> 271.5 mm, vias 0 -> 3
- net col10: track 0.00 -> 239.8 mm, vias 0 -> 3
- net col11: track 0.00 -> 235.8 mm, vias 0 -> 7
- net row2: track 0.00 -> 230.0 mm, vias 0 -> 3
- net row1: track 0.00 -> 229.8 mm, vias 0 -> 4
- net col8: track 0.00 -> 228.0 mm, vias 0 -> 1
- net col9: track 0.00 -> 215.3 mm, vias 0 -> 1
- net col7: track 0.00 -> 203.7 mm, vias 0 -> 1
- net row3: track 0.00 -> 197.7 mm, vias 0 -> 2
- net col6: track 0.00 -> 169.8 mm, vias 0 -> 5
- net col5: track 0.00 -> 168.2 mm, vias 0 -> 5
- net col4: track 0.00 -> 161.7 mm, vias 0 -> 3
- net col3: track 0.00 -> 130.4 mm, vias 0 -> 2
- net +3V3: track 0.00 -> 102.4 mm, vias 0 -> 6
- net col2: track 0.00 -> 77.4 mm
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- added copper zone on B.Cu, net +1V1
- added copper zone on B.Cu, net +3V3
- added copper zone on B.Cu, net GND
- added copper zone on F.Cu, net GND
Other:
- board size 228.6 x 76.2 mm -> 228.6 x 77.7 mm
